Commit message: モデルにendtipを追加

File: crane_plus_description/urdf/crane_plus.urdf.xacro (robot description, xacro)
@@ -22,4 +22,6 @@
   <xacro:arg name="gz_control_config_package" default="" />
   <xacro:arg name="gz_control_config_file_path" default="" />
+  <xacro:arg name="endtip_offset_xyz" default="0 0 0" />
+  <xacro:arg name="endtip_offset_rpy" default="0 0 0" />
   <!-- Link to provide the location reference for the arm -->
   <link name="base_link"/>
@@ -36,4 +38,5 @@
   <xacro:property name="NAME_LINK_4" value="crane_plus_link4"/>
   <xacro:property name="NAME_LINK_HAND" value="crane_plus_link_hand"/>
+  <xacro:property name="NAME_LINK_ENDTIP" value="crane_plus_link_endtip"/>
   <xacro:property name="NAME_JOINT_BASE" value="crane_plus_joint_base"/>
   <xacro:property name="NAME_JOINT_1" value="crane_plus_joint1"/>
@@ -42,4 +45,5 @@
   <xacro:property name="NAME_JOINT_4" value="crane_plus_joint4"/>
   <xacro:property name="NAME_JOINT_HAND" value="crane_plus_joint_hand"/>
+  <xacro:property name="NAME_JOINT_ENDTIP" value="crane_plus_joint_endtip"/>
   <xacro:property name="M_PI" value="3.14159"/>
   <xacro:property name="TO_RADIAN" value="${M_PI / 180.0}"/>
@@ -64,4 +68,5 @@
     name_link_4="${NAME_LINK_4}"
     name_link_hand="${NAME_LINK_HAND}"
+    name_link_endtip="${NAME_LINK_ENDTIP}"
     name_joint_base="${NAME_JOINT_BASE}"
     name_joint_1="${NAME_JOINT_1}"
@@ -70,4 +75,5 @@
     name_joint_4="${NAME_JOINT_4}"
     name_joint_hand="${NAME_JOINT_HAND}"
+    name_joint_endtip="${NAME_JOINT_ENDTIP}"
     joints_vlimit="${JOINT_VELOCITY_LIMIT}"
     joint_1_lower_limit="${JOINT_1_LOWER_LIMIT}"
@@ -81,5 +87,7 @@
     joint_hand_lower_limit="${JOINT_HAND_LOWER_LIMIT}"
     joint_hand_upper_limit="${JOINT_HAND_UPPER_LIMIT}"
-    use_camera="$(arg use_camera)">
+    use_camera="$(arg use_camera)"
+    endtip_offset_xyz="$(arg endtip_offset_xyz)"
+    endtip_offset_rpy="$(arg endtip_offset_rpy)">
     <origin xyz="0 0 0"/>
   </xacro:crane_plus>

File: crane_plus_description/urdf/crane_plus.xacro (robot description, xacro)
@@ -41,4 +41,5 @@
               name_link_4
               name_link_hand
+              name_link_endtip
               name_joint_base
               name_joint_1
@@ -47,4 +48,5 @@
               name_joint_4
               name_joint_hand
+              name_joint_endtip
               joints_vlimit
               joint_1_lower_limit
@@ -59,4 +61,6 @@
               joint_hand_upper_limit
               use_camera
+              endtip_offset_xyz
+              endtip_offset_rpy
               *origin">
     <joint name="${name_joint_base}" type="fixed">
@@ -268,4 +272,11 @@
       </inertial>
     </link>
+    <!-- Tool Center Point for MoveIt -->
+    <joint name="${name_joint_endtip}" type="fixed">
+      <origin xyz="${endtip_offset_xyz}" rpy="${endtip_offset_rpy}"/>
+      <parent link="${name_link_4}"/>
+      <child link="${name_link_endtip}"/>
+    </joint>
+    <link name="${name_link_endtip}"/>
     <!-- camera -->
     <xacro:if value="$(arg use_camera)">
